File: CH2_Esquema_y_PCB/Esquema_y_PCB.kicad_sch (KiCad schematic)
At the start: 43 parts, among them Q1 BC547, Q10 BC857, Q2 BC547, Q3 BC547, Q4 BC547, Q5 IRF9Z34N, Q7 BC547, Q9 BC857, U1 TL431LP, U2 LM358

Commit message: Rehecho PCB
Parts:
- added unit 2 of U2
- C2, C3: footprint Capacitor_THT:C_Disc_D5.0mm_W2.5mm_P5.00mm -> Capacitor_THT:C_Disc_D7.5mm_W5.0mm_P7.50mm
- Q1, Q10, Q2, Q3, Q4, Q7, Q9, U1: footprint Package_TO_SOT_THT:TO-92_Inline -> Package_TO_SOT_THT:TO-92_Wide
- R11, R15, R16, R3, R4, R5, R6, R7, R8, R9, RF1: footprint Resistor_THT:R_Axial_DIN0204_L3.6mm_D1.6mm_P5.08mm_Horizontal -> Resistor_THT:R_Axial_DIN0207_L6.3mm_D2.5mm_P10.16mm_Horizontal
- RS1: footprint Resistor_THT:R_Axial_DIN0414_L11.9mm_D4.5mm_P15.24mm_Horizontal -> Resistor_THT:R_Axial_Power_L20.0mm_W6.4mm_P25.40mm
Connections:
- net GND: now also U2.5 (+), U2.6 (-), U2.7
- net drain: now also Q5.2 (D); no longer Q5.1 (D)
- net gate: now also Q5.1 (G); no longer Q5.2 (G)
- net at R13.2: now also Q9.1 (E); no longer Q9.2 (E)
- net at Q10.3 (C), Q2.1 (C): now also Q10.2 (B), Q9.2 (B); no longer Q10.1 (B), Q9.1 (B)
- net at R14.2: now also Q10.1 (E); no longer Q10.2 (E)
