File: CH2_Esquema_y_PCB/Esquema_y_PCB.kicad_pcb (KiCad board)
At the start: 2 copper layers, 140.1 x 79.8 mm, 44 parts, among them Q1 BC547, Q10 BC857, Q2 BC547, Q3 BC547, Q4 BC547, Q5 IRF9Z34N, Q7 BC547, Q9 BC857, U1 TL431LP, U2 LM358

Commit message: Add files via upload
Parts:
- R11, R15, R16, R3, R4, R5, R6, R7, R8, R9, RF1: footprint Resistor_THT:R_Axial_DIN0204_L3.6mm_D1.6mm_P5.08mm_Horizontal -> Resistor_THT:R_Axial_DIN0207_L6.3mm_D2.5mm_P10.16mm_Horizontal
- moved JP10 6.50 mm to (148.1, 96.2)
- moved JP11 5.50 mm to (137.1, 95.2)
- moved R8 5.31 mm to (137.0, 89.1)
- moved R6 5.31 mm to (166.5, 89.1)
- moved R7 5.31 mm to (148.0, 89.0)
- moved R5 5.27 mm to (157.5, 89.0)
- moved R3 5.04 mm to (99.6, 92.6)
- moved R2 4.32 mm to (128.8, 99.0)
- moved R4 4.08 mm to (64.0, 82.4)
- moved JP7 3.59 mm to (89.8, 75.0), turned to 0 degrees
- moved Q4 3.46 mm to (68.5, 93.5)
- moved R1 2.72 mm to (94.0, 85.4)
- moved RF1 2.46 mm to (144.6, 59.0)
- moved R9 2.35 mm to (128.1, 86.1)
- moved JP12 2.25 mm to (128.0, 92.0)
Routing:
- net /gate: track 195.6 -> 205.6 mm
- net Net-(JP7-A): track 70.0 -> 63.4 mm
- net /out: track 57.8 -> 64.2 mm
- net Net-(JP7-B): track 23.0 -> 28.6 mm
- net Net-(Q3-B): track 27.1 -> 23.1 mm
- net /drain: track 187.1 -> 184.5 mm
- net Net-(JP8-A): track 28.9 -> 31.0 mm
- net Net-(U2A-+): track 64.1 -> 66.1 mm
- net GND: track 2.09 -> 3.45 mm
- net Net-(Q7-B): track 7.80 -> 9.00 mm
- net Net-(JP10-B): track 3.56 -> 4.74 mm

Commit message: Add files via upload
Parts:
- RS1: footprint Resistor_THT:R_Axial_DIN0414_L11.9mm_D4.5mm_P15.24mm_Horizontal -> Resistor_THT:R_Axial_Power_L20.0mm_W6.4mm_P25.40mm
- moved R11 17.8 mm to (126.5, 67.6)
- moved RS1 12.6 mm to (109.5, 55.6)
- moved JP9 3.49 mm to (102.2, 57.5), turned to 180 degrees
Routing:
- net Net-(U2A--): track 59.8 -> 45.6 mm
- net /gate: track 205.6 -> 211.1 mm
- net Net-(JP9-A): track 3.63 -> 8.12 mm
- net /out: track 64.2 -> 60.0 mm

Commit message: Add files via upload
Parts:
- C2, C3: footprint Capacitor_THT:C_Disc_D5.0mm_W2.5mm_P5.00mm -> Capacitor_THT:C_Disc_D7.5mm_W5.0mm_P7.50mm
- Q1, Q10, Q2, Q3, Q4, Q7, Q9, U1: footprint Package_TO_SOT_THT:TO-92_Inline -> Package_TO_SOT_THT:TO-92_Wide
- moved G*** 112.4 mm to (169.1, 108.2)
- moved JP10 49.6 mm to (122.1, 54.0), turned to -90 degrees
- moved R7 38.1 mm to (122.1, 61.0), turned to -90 degrees
- moved R16 35.2 mm to (148.0, 41.8), turned to -90 degrees
- moved R6 17.7 mm to (148.8, 89.0)
- moved Q7 14.5 mm to (151.5, 58.3)
- moved V1 14.3 mm to (50.8, 41.0), turned to -90 degrees
- moved R5 13.6 mm to (143.9, 88.9)
- moved Q10 11.8 mm to (63.7, 59.0), turned to -90 degrees
- moved C3 11.6 mm to (96.5, 61.5)
- moved R15 11.0 mm to (170.5, 49.4), turned to -90 degrees
- moved C2 9.83 mm to (96.8, 80.9), turned to 0 degrees
- moved R3 8.96 mm to (93.7, 85.8), turned to 0 degrees
- moved U1 8.57 mm to (60.1, 80.7), turned to 90 degrees
- moved R1 7.20 mm to (94.2, 92.6)
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Connections:
- Q10 pad 1: Net-(Q10-B) -> Net-(Q10-E)
- Q10 pad 2: Net-(Q10-E) -> Net-(Q10-B)
- Q5 pad 1: /drain -> /gate
- Q5 pad 2: /gate -> /drain
- Q9 pad 1: Net-(Q10-B) -> Net-(Q9-E)
- Q9 pad 2: Net-(Q9-E) -> Net-(Q10-B)
- U2 pad 5: (no net) -> GND
- U2 pad 6: (no net) -> GND
- U2 pad 7: (no net) -> GND
Routing:
- net /drain: track 184.5 -> 55.4 mm
- net /gate: track 211.1 -> 150.2 mm
- net /in: track 109.0 -> 157.4 mm
- net VCC: track 376.1 -> 346.5 mm
- net Net-(Q10-B): track 19.3 -> 40.9 mm
- net Net-(JP14-A): track 7.93 -> 24.4 mm
- net Net-(JP7-A): track 63.4 -> 47.0 mm
- net Net-(JP8-B): track 5.79 -> 16.0 mm
- net Net-(Q7-B): track 9.00 -> 18.1 mm
- net Net-(U2A-+): track 66.1 -> 71.7 mm
- net Net-(Q10-E): track 5.78 -> 10.9 mm
- net Net-(Q3-C): track 15.4 -> 11.4 mm
- net GND: track 3.45 -> 0.00 mm
- net Net-(Q3-B): track 23.1 -> 26.5 mm
- net Net-(JP9-A): track 8.12 -> 5.04 mm
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Other:
- board size 140.1 x 79.8 mm -> 143.4 x 79.8 mm
- board text added: "[TA 138] TDCE - GRUPO 2 - V3.0 -"
- board text removed: "[TA 138] TDCE - GRUPO 2 - V2.0 ROZENBERG, FERRUA, CHAPARRO Y CAMPISI"
