File: CH3_Esquema_y_PCB/Esquema_y_PCB.kicad_sch (KiCad schematic)
At the start: 44 parts, among them Q1 BC547, Q10 BC857, Q2 BC547, Q3 BC547, Q4 BC547, Q5 IRF9Z34N, Q7 BC547, Q9 BC857, U1 TL431LP, U2 LM358

Commit message: Add files via upload
Parts:
- removed Q7: BC547, Package_TO_SOT_THT:TO-92_Wide, symbol Transistor_BJT:BC547
- removed R1: 10k, Resistor_THT:R_Axial_DIN0207_L6.3mm_D2.5mm_P10.16mm_Horizontal, symbol Device:R
- added Q11: BC557, Package_TO_SOT_THT:TO-92_Wide, symbol Transistor_BJT:BC857
- added RV1: R_Potentiometer, Potentiometer_THT:Potentiometer_Bourns_3266W_Vertical, symbol Device:R_Potentiometer
- C3: footprint Capacitor_THT:C_Disc_D7.5mm_W5.0mm_P7.50mm -> Capacitor_THT:C_Disc_D5.0mm_W2.5mm_P5.00mm
- C4: footprint Capacitor_THT:C_Disc_D5.0mm_W2.5mm_P5.00mm -> Capacitor_THT:C_Disc_D8.0mm_W5.0mm_P10.00mm
- Q10, Q9: value BC857 -> BC557
- R10: footprint Resistor_THT:R_Axial_DIN0207_L6.3mm_D2.5mm_P10.16mm_Horizontal -> Resistor_THT:R_Axial_DIN0207_L6.3mm_D2.5mm_P15.24mm_Horizontal
- R16, R7: footprint Resistor_THT:R_Axial_DIN0207_L6.3mm_D2.5mm_P15.24mm_Horizontal -> Resistor_THT:R_Axial_DIN0207_L6.3mm_D2.5mm_P10.16mm_Horizontal
Connections:
- net GND: now also RV1.1, RV1.2
- net at C4.1, R5.2, R6.2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: now also U2.2 (-); no longer U2.3 (+)
- net at R16.2: now also Q11.1 (E)
- net at C2.1, JP7.2 (B), R3.1: now also RV1.3
- net at R10.2, R11.1, R8.2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: now also U2.3 (+); no longer U2.2 (-)
- net at R15.2: now also Q11.2 (B)
- net at JP14.1 (A): now also Q11.3 (C)
Other:
- moved on the sheet: C3

Commit message: Add files via upload
Parts:
- removed JP10, JP11, JP12, JP13, JP14: Jumper_2_Bridged, TestPoint:TestPoint_2Pads_Pitch2.54mm_Drill0.8mm, symbol Jumper:Jumper_2_Bridged
- removed RV1: R_Potentiometer, Potentiometer_THT:Potentiometer_Bourns_3266W_Vertical, symbol Device:R_Potentiometer
- added R7: 5k1, Resistor_THT:R_Axial_DIN0207_L6.3mm_D2.5mm_P10.16mm_Horizontal, symbol Device:R
- C2: value 820p -> 1.2n
- CF1: renamed from C4; footprint Capacitor_THT:C_Disc_D8.0mm_W5.0mm_P10.00mm -> Capacitor_THT:C_Disc_D5.0mm_W2.5mm_P5.00mm
- R1: renamed from R17; value 2k2 -> 1k
- R2: renamed from R12; value 2k2 -> 1k
- R6: renamed from R3; value 10k -> 5k1
- renumbered JP15 to JP1, JP7 to JP2, JP9 to JP3, JP8 to JP4, Q5 to MOS1, Q9 to Q5, Q10 to Q6, Q11 to Q7, R7 to R10, R8 to R11, R9 to R12, R10 to R13, R11 to R14, R4 to R3, R13 to R4, R14 to R5, R5 to R8, R6 to R9, R2 to RL1
Connections:
- net GND: now also R7.1
- net VB: now also Q7.3 (C)
- net drain: now also R10.1
- net in: now also R13.1
- net out: now also R11.1, R12.1
- net at C2.1, JP2.2 (B), R6.1: now also R7.2
Other:
- moved on the sheet: C1, C3, JP2, JP3, JP4, R15
